Commit message: update urdf

File: g1_description/urdf/g1_body29_hand14.urdf (robot description, URDF)
Before this commit: robot g1_29dof_lock_waist_rev_1_0, 39 links, 38 joints
Links:
- removed link left_rubber_hand
- removed link right_rubber_hand
- added link left_hand_index_0_link, mass 0.05885070; collision mesh filename=meshes/left_hand_index_0_link.STL; visual mesh filename=meshes/left_hand_index_0_link.STL
- added link left_hand_index_1_link, mass 0.02030626; collision mesh filename=meshes/left_hand_index_1_link.STL; visual mesh filename=meshes/left_hand_index_1_link.STL
- added link left_hand_middle_0_link, mass 0.05885070; collision mesh filename=meshes/left_hand_middle_0_link.STL; visual mesh filename=meshes/left_hand_middle_0_link.STL
- added link left_hand_middle_1_link, mass 0.02030626; collision mesh filename=meshes/left_hand_middle_1_link.STL; visual mesh filename=meshes/left_hand_middle_1_link.STL
- added link left_hand_palm_link, mass 0.37283854; collision mesh filename=meshes/left_hand_palm_link.STL; visual mesh filename=meshes/left_hand_palm_link.STL
- added link left_hand_thumb_0_link, mass 0.08623657; collision mesh filename=meshes/left_hand_thumb_0_link.STL; visual mesh filename=meshes/left_hand_thumb_0_link.STL
- added link left_hand_thumb_1_link, mass 0.05885070; collision box size=0.02 0.03 0.02; visual mesh filename=meshes/left_hand_thumb_1_link.STL
- added link left_hand_thumb_2_link, mass 0.02030626; collision mesh filename=meshes/left_hand_thumb_2_link.STL; visual mesh filename=meshes/left_hand_thumb_2_link.STL
- added link right_hand_index_0_link, mass 0.05885070; collision mesh filename=meshes/right_hand_index_0_link.STL; visual mesh filename=meshes/right_hand_index_0_link.STL
- added link right_hand_index_1_link, mass 0.02030626; collision mesh filename=meshes/right_hand_index_1_link.STL; visual mesh filename=meshes/right_hand_index_1_link.STL
- added link right_hand_middle_0_link, mass 0.05885070; collision mesh filename=meshes/right_hand_middle_0_link.STL; visual mesh filename=meshes/right_hand_middle_0_link.STL
- added link right_hand_middle_1_link, mass 0.02030626; collision mesh filename=meshes/right_hand_middle_1_link.STL; visual mesh filename=meshes/right_hand_middle_1_link.STL
- added link right_hand_palm_link, mass 0.37283854; collision mesh filename=meshes/right_hand_palm_link.STL; visual mesh filename=meshes/right_hand_palm_link.STL
- added link right_hand_thumb_0_link, mass 0.08623657; collision mesh filename=meshes/right_hand_thumb_0_link.STL; visual mesh filename=meshes/right_hand_thumb_0_link.STL
- added link right_hand_thumb_1_link, mass 0.05885070; collision box size=0.02 0.03 0.02; visual mesh filename=meshes/right_hand_thumb_1_link.STL
- added link right_hand_thumb_2_link, mass 0.02030626; collision mesh filename=meshes/right_hand_thumb_2_link.STL; visual mesh filename=meshes/right_hand_thumb_2_link.STL
- added link world
Joints:
- added joint floating_base_joint: type floating, parent world, child pelvis
- added joint left_hand_index_0_joint: type revolute, parent left_hand_palm_link, child left_hand_index_0_link, origin xyz=0.0777 0.0016 0.0285 rpy=0 0 0, axis 0 0 1, limit lower=-1.57079632 upper=0 effort=1.4 velocity=12
- added joint left_hand_index_1_joint: type revolute, parent left_hand_index_0_link, child left_hand_index_1_link, origin xyz=0.0458 0 0 rpy=0 0 0, axis 0 0 1, limit lower=-1.74532925 upper=0 effort=1.4 velocity=12
- added joint left_hand_middle_0_joint: type revolute, parent left_hand_palm_link, child left_hand_middle_0_link, origin xyz=0.0777 0.0016 -0.0285 rpy=0 0 0, axis 0 0 1, limit lower=-1.57079632 upper=0 effort=1.4 velocity=12
- added joint left_hand_middle_1_joint: type revolute, parent left_hand_middle_0_link, child left_hand_middle_1_link, origin xyz=0.0458 0 0 rpy=0 0 0, axis 0 0 1, limit lower=-1.74532925 upper=0 effort=1.4 velocity=12
- added joint left_hand_thumb_0_joint: type revolute, parent left_hand_palm_link, child left_hand_thumb_0_link, origin xyz=0.0255 0 0 rpy=0 0 0, axis 0 1 0, limit lower=-1.04719755 upper=1.04719755 effort=2.45 velocity=6.857
- added joint left_hand_thumb_1_joint: type revolute, parent left_hand_thumb_0_link, child left_hand_thumb_1_link, origin xyz=-0.0025 -0.0193 0 rpy=0 0 0, axis 0 0 1, limit lower=-0.72431163 upper=1.04719755 effort=1.4 velocity=12
- added joint left_hand_thumb_2_joint: type revolute, parent left_hand_thumb_1_link, child left_hand_thumb_2_link, origin xyz=0 -0.0458 0 rpy=0 0 0, axis 0 0 1, limit lower=0 upper=1.74532925 effort=1.4 velocity=12
- added joint right_hand_index_0_joint: type revolute, parent right_hand_palm_link, child right_hand_index_0_link, origin xyz=0.0777 -0.0016 0.0285 rpy=0 0 0, axis 0 0 1, limit lower=0 upper=1.57079632 effort=1.4 velocity=12
- added joint right_hand_index_1_joint: type revolute, parent right_hand_index_0_link, child right_hand_index_1_link, origin xyz=0.0458 0 0 rpy=0 0 0, axis 0 0 1, limit lower=0 upper=1.74532925 effort=1.4 velocity=12
- added joint right_hand_middle_0_joint: type revolute, parent right_hand_palm_link, child right_hand_middle_0_link, origin xyz=0.0777 -0.0016 -0.0285 rpy=0 0 0, axis 0 0 1, limit lower=0 upper=1.57079632 effort=1.4 velocity=12
- added joint right_hand_middle_1_joint: type revolute, parent right_hand_middle_0_link, child right_hand_middle_1_link, origin xyz=0.0458 0 0 rpy=0 0 0, axis 0 0 1, limit lower=0 upper=1.74532925 effort=1.4 velocity=12
- added joint right_hand_thumb_0_joint: type revolute, parent right_hand_palm_link, child right_hand_thumb_0_link, origin xyz=0.0255 0 0 rpy=0 0 0, axis 0 1 0, limit lower=-1.04719755 upper=1.04719755 effort=2.45 velocity=6.857
- added joint right_hand_thumb_1_joint: type revolute, parent right_hand_thumb_0_link, child right_hand_thumb_1_link, origin xyz=-0.0025 0.0193 0 rpy=0 0 0, axis 0 0 1, limit lower=-1.04719755 upper=0.72431163 effort=1.4 velocity=12
- added joint right_hand_thumb_2_joint: type revolute, parent right_hand_thumb_1_link, child right_hand_thumb_2_link, origin xyz=0 0.0458 0 rpy=0 0 0, axis 0 0 1, limit lower=-1.74532925 upper=0 effort=1.4 velocity=12
- joint left_hand_palm_joint: child left_rubber_hand -> left_hand_palm_link
- joint right_hand_palm_joint: child right_rubber_hand -> right_hand_palm_link
- joint waist_pitch_joint: type fixed -> revolute
- joint waist_roll_joint: type fixed -> revolute

Commit message: added mid360 launch and fix transform

File: g1_description/urdf/g1_body29_hand14.urdf (robot description, URDF)
Before this commit: robot g1, 54 links, 53 joints
Joints:
- joint mid360_joint: origin xyz=0.0002835 0.00003 0.41618 rpy=0 0.04014257279586953 0 -> xyz=0.0002835 0.00003 0.41618 rpy=0 3.14159 3.14159

Commit message: update the configs

File: g1_description/urdf/g1_body29_hand14.urdf (robot description, URDF)
Before this commit: robot g1, 54 links, 53 joints
Joints:
- joint mid360_joint: origin xyz=0.0002835 0.00003 0.41618 rpy=0 3.14159 3.14159 -> xyz=0.0002835 0.00003 0.41618 rpy=-3.1415927 0.0401426 0

Commit message: update urdf mesh filename and collision

File: g1_description/urdf/g1_body29_hand14.urdf (robot description, URDF)
Before this commit: robot g1, 54 links, 53 joints
Links:
- link head_link: geometry collision mesh filename=package://g1_description/urdf/meshes/head_link.STL; visual mesh filename=package://g1_description/urdf/meshes/head_link.STL
- link left_ankle_pitch_link: geometry collision mesh filename=package://g1_description/urdf/meshes/left_ankle_pitch_link.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; visual mesh filename=package://g1_description/urdf/meshes/left_ankle_pitch_link.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
- link left_ankle_roll_link: geometry collision mesh filename=package://g1_description/urdf/meshes/left_ankle_roll_link.S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; visual mesh filename=package://g1_description/urdf/meshes/left_ankle_roll_link.S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
- link left_elbow_link: geometry collision mesh filename=package://g1_description/urdf/meshes/left_elbow_link.STL; visual mesh filename=package://g1_description/urdf/meshes/left_elbow_link.STL
- link left_hand_index_0_link: geometry collision mesh filename=package://g1_description/urdf/meshes/left_hand_index_0_link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; visual mesh filename=package://g1_description/urdf/meshes/left_hand_index_0_link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
- link left_hand_index_1_link: geometry collision mesh filename=package://g1_description/urdf/meshes/left_hand_index_1_link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; visual mesh filename=package://g1_description/urdf/meshes/left_hand_index_1_link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
- link left_hand_middle_0_link: geometry collision mesh filename=package://g1_description/urdf/meshes/left_hand_middle_0_lin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; visual mesh filename=package://g1_description/urdf/meshes/left_hand_middle_0_lin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
- link left_hand_middle_1_link: geometry collision mesh filename=package://g1_description/urdf/meshes/left_hand_middle_1_lin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; visual mesh filename=package://g1_description/urdf/meshes/left_hand_middle_1_lin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
- link left_hand_palm_link: geometry collision mesh filename=package://g1_description/urdf/meshes/left_hand_palm_link.STL; visual mesh filename=package://g1_description/urdf/meshes/left_hand_palm_link.STL
- link left_hand_thumb_0_link: geometry collision mesh filename=package://g1_description/urdf/meshes/left_hand_thumb_0_link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; visual mesh filename=package://g1_description/urdf/meshes/left_hand_thumb_0_link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
- link left_hand_thumb_1_link: geometry collision mesh filename=package://g1_description/urdf/meshes/left_hand_thumb_1_link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; visual mesh filename=package://g1_description/urdf/meshes/left_hand_thumb_1_link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
- link left_hand_thumb_2_link: geometry collision mesh filename=package://g1_description/urdf/meshes/left_hand_thumb_2_link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; visual mesh filename=package://g1_description/urdf/meshes/left_hand_thumb_2_link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
- link left_hip_pitch_link: geometry collision mesh filename=package://g1_description/urdf/meshes/left_hip_pitch_link.STL; visual mesh filename=package://g1_description/urdf/meshes/left_hip_pitch_link.STL
- link left_hip_roll_link: geometry collision mesh filename=package://g1_description/urdf/meshes/left_hip_roll_link.STL; visual mesh filename=package://g1_description/urdf/meshes/left_hip_roll_link.STL
- link left_hip_yaw_link: geometry collision mesh filename=package://g1_description/urdf/meshes/left_hip_yaw_link.STL; visual mesh filename=package://g1_description/urdf/meshes/left_hip_yaw_link.STL
- link left_knee_link: geometry collision mesh filename=package://g1_description/urdf/meshes/left_knee_link.STL; visual mesh filename=package://g1_description/urdf/meshes/left_knee_link.STL
- link left_shoulder_pitch_link: geometry collision mesh filename=package://g1_description/urdf/meshes/left_shoulder_pitch_li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; visual mesh filename=package://g1_description/urdf/meshes/left_shoulder_pitch_li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
- link left_shoulder_roll_link: geometry collision mesh filename=package://g1_description/urdf/meshes/left_shoulder_roll_lin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; visual mesh filename=package://g1_description/urdf/meshes/left_shoulder_roll_lin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
- link left_shoulder_yaw_link: geometry collision mesh filename=package://g1_description/urdf/meshes/left_shoulder_yaw_link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; visual mesh filename=package://g1_description/urdf/meshes/left_shoulder_yaw_link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
- link left_wrist_pitch_link: geometry collision mesh filename=package://g1_description/urdf/meshes/left_wrist_pitch_link.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; visual mesh filename=package://g1_description/urdf/meshes/left_wrist_pitch_link.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
- link left_wrist_roll_link: geometry collision mesh filename=package://g1_description/urdf/meshes/left_wrist_roll_link.S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; visual mesh filename=package://g1_description/urdf/meshes/left_wrist_roll_link.S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
- link left_wrist_yaw_link: geometry collision mesh filename=package://g1_description/urdf/meshes/left_wrist_yaw_link.STL; visual mesh filename=package://g1_description/urdf/meshes/left_wrist_yaw_link.STL
- link logo_link: geometry collision mesh filename=package://g1_description/urdf/meshes/logo_link.STL; visual mesh filename=package://g1_description/urdf/meshes/logo_link.STL
- link pelvis: geometry collision mesh filename=package://g1_description/urdf/meshes/pelvis.STL; visual mesh filename=package://g1_description/urdf/meshes/pelvis.STL
- link pelvis_contour_link: geometry collision mesh filename=package://g1_description/urdf/meshes/pelvis_contour_link.STL; visual mesh filename=package://g1_description/urdf/meshes/pelvis_contour_link.STL
- link right_ankle_pitch_link: geometry collision mesh filename=package://g1_description/urdf/meshes/right_ankle_pitch_link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; visual mesh filename=package://g1_description/urdf/meshes/right_ankle_pitch_link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
- link right_ankle_roll_link: geometry collision mesh filename=package://g1_description/urdf/meshes/right_ankle_roll_link.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; visual mesh filename=package://g1_description/urdf/meshes/right_ankle_roll_link.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
- link right_elbow_link: geometry collision mesh filename=package://g1_description/urdf/meshes/right_elbow_link.STL; visual mesh filename=package://g1_description/urdf/meshes/right_elbow_link.STL
- link right_hand_index_0_link: geometry collision mesh filename=package://g1_description/urdf/meshes/right_hand_index_0_lin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; visual mesh filename=package://g1_description/urdf/meshes/right_hand_index_0_lin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
- link right_hand_index_1_link: geometry collision mesh filename=package://g1_description/urdf/meshes/right_hand_index_1_lin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; visual mesh filename=package://g1_description/urdf/meshes/right_hand_index_1_lin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
- link right_hand_middle_0_link: geometry collision mesh filename=package://g1_description/urdf/meshes/right_hand_middle_0_li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; visual mesh filename=package://g1_description/urdf/meshes/right_hand_middle_0_li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
- link right_hand_middle_1_link: geometry collision mesh filename=package://g1_description/urdf/meshes/right_hand_middle_1_li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; visual mesh filename=package://g1_description/urdf/meshes/right_hand_middle_1_li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
- link right_hand_palm_link: geometry collision mesh filename=package://g1_description/urdf/meshes/right_hand_palm_link.S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; visual mesh filename=package://g1_description/urdf/meshes/right_hand_palm_link.S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
- link right_hand_thumb_0_link: geometry collision mesh filename=package://g1_description/urdf/meshes/right_hand_thumb_0_lin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; visual mesh filename=package://g1_description/urdf/meshes/right_hand_thumb_0_lin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
- link right_hand_thumb_1_link: geometry collision mesh filename=package://g1_description/urdf/meshes/right_hand_thumb_1_lin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; visual mesh filename=package://g1_description/urdf/meshes/right_hand_thumb_1_lin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
- link right_hand_thumb_2_link: geometry collision mesh filename=package://g1_description/urdf/meshes/right_hand_thumb_2_lin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; visual mesh filename=package://g1_description/urdf/meshes/right_hand_thumb_2_lin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
- link right_hip_pitch_link: geometry collision mesh filename=package://g1_description/urdf/meshes/right_hip_pitch_link.S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; visual mesh filename=package://g1_description/urdf/meshes/right_hip_pitch_link.S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
- link right_hip_roll_link: geometry collision mesh filename=package://g1_description/urdf/meshes/right_hip_roll_link.STL; visual mesh filename=package://g1_description/urdf/meshes/right_hip_roll_link.STL
- link right_hip_yaw_link: geometry collision mesh filename=package://g1_description/urdf/meshes/right_hip_yaw_link.STL; visual mesh filename=package://g1_description/urdf/meshes/right_hip_yaw_link.STL
- link right_knee_link: geometry collision mesh filename=package://g1_description/urdf/meshes/right_knee_link.STL; visual mesh filename=package://g1_description/urdf/meshes/right_knee_link.STL
- link right_shoulder_pitch_link: geometry collision mesh filename=package://g1_description/urdf/meshes/right_shoulder_pitch_l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; visual mesh filename=package://g1_description/urdf/meshes/right_shoulder_pitch_l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
- link right_shoulder_roll_link: geometry collision mesh filename=package://g1_description/urdf/meshes/right_shoulder_roll_li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; visual mesh filename=package://g1_description/urdf/meshes/right_shoulder_roll_li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
- link right_shoulder_yaw_link: geometry collision mesh filename=package://g1_description/urdf/meshes/right_shoulder_yaw_lin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; visual mesh filename=package://g1_description/urdf/meshes/right_shoulder_yaw_lin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
- link right_wrist_pitch_link: geometry collision mesh filename=package://g1_description/urdf/meshes/right_wrist_pitch_link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; visual mesh filename=package://g1_description/urdf/meshes/right_wrist_pitch_link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
- link right_wrist_roll_link: geometry collision mesh filename=package://g1_description/urdf/meshes/right_wrist_roll_link.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; visual mesh filename=package://g1_description/urdf/meshes/right_wrist_roll_link.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
- link right_wrist_yaw_link: geometry collision mesh filename=package://g1_description/urdf/meshes/right_wrist_yaw_link.S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; visual mesh filename=package://g1_description/urdf/meshes/right_wrist_yaw_link.S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
- link torso_link: geometry collision mesh filename=package://g1_description/urdf/meshes/torso_link_rev_1_0.STL; visual mesh filename=package://g1_description/urdf/meshes/torso_link_rev_1_0.STL
- link waist_roll_link: geometry collision mesh filename=package://g1_description/urdf/meshes/waist_roll_link_rev_1_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; visual mesh filename=package://g1_description/urdf/meshes/waist_roll_link_rev_1_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
- link waist_yaw_link: geometry collision mesh filename=package://g1_description/urdf/meshes/waist_yaw_link_rev_1_0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; visual mesh filename=package://g1_description/urdf/meshes/waist_yaw_link_rev_1_0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
