Commit message: added inspire hand into urdf and xml

File: g1_description/urdf/g1_body29_hand14.urdf (robot description, URDF)
Before this commit: robot g1, 54 links, 53 joints
Links:
- removed link left_hand_index_0_link
- removed link left_hand_index_1_link
- removed link left_hand_middle_0_link
- removed link left_hand_middle_1_link
- removed link left_hand_palm_link
- removed link left_hand_thumb_0_link
- removed link left_hand_thumb_1_link
- removed link left_hand_thumb_2_link
- removed link right_hand_index_0_link
- removed link right_hand_index_1_link
- removed link right_hand_middle_0_link
- removed link right_hand_middle_1_link
- removed link right_hand_palm_link
- removed link right_hand_thumb_0_link
- removed link right_hand_thumb_1_link
- removed link right_hand_thumb_2_link
- added link L_hand_base_link, mass 0.14143; collision mesh filename=package://g1_description/urdf/meshes/L_hand_base_link.STL; visual mesh filename=package://g1_description/urdf/meshes/L_hand_base_link.STL
- added link L_index_intermediate, mass 0.0045682; collision mesh filename=package://g1_description/urdf/meshes/Link16_L.STL; visual mesh filename=package://g1_description/urdf/meshes/Link16_L.STL
- added link L_index_proximal, mass 0.0042405; collision mesh filename=package://g1_description/urdf/meshes/Link15_L.STL; visual mesh filename=package://g1_description/urdf/meshes/Link15_L.STL
- added link L_index_tip; visual sphere radius=0.005
- added link L_middle_intermediate, mass 0.0050397; collision mesh filename=package://g1_description/urdf/meshes/Link18_L.STL; visual mesh filename=package://g1_description/urdf/meshes/Link18_L.STL
- added link L_middle_proximal, mass 0.0042405; collision mesh filename=package://g1_description/urdf/meshes/Link17_L.STL; visual mesh filename=package://g1_description/urdf/meshes/Link17_L.STL
- added link L_middle_tip; visual sphere radius=0.005
- added link L_pinky_intermediate, mass 0.0036036; collision mesh filename=package://g1_description/urdf/meshes/Link22_L.STL; visual mesh filename=package://g1_description/urdf/meshes/Link22_L.STL
- added link L_pinky_proximal, mass 0.0042405; collision mesh filename=package://g1_description/urdf/meshes/Link21_L.STL; visual mesh filename=package://g1_description/urdf/meshes/Link21_L.STL
- added link L_pinky_tip; visual sphere radius=0.005
- added link L_ring_intermediate, mass 0.0045682; collision mesh filename=package://g1_description/urdf/meshes/Link20_L.STL; visual mesh filename=package://g1_description/urdf/meshes/Link20_L.STL
- added link L_ring_proximal, mass 0.0042405; collision mesh filename=package://g1_description/urdf/meshes/Link19_L.STL; visual mesh filename=package://g1_description/urdf/meshes/Link19_L.STL
- added link L_ring_tip; visual sphere radius=0.005
- added link L_thumb_distal, mass 0.003344; collision mesh filename=package://g1_description/urdf/meshes/Link14_L.STL; visual mesh filename=package://g1_description/urdf/meshes/Link14_L.STL
- added link L_thumb_intermediate, mass 0.0037844; collision mesh filename=package://g1_description/urdf/meshes/Link13_L.STL; visual mesh filename=package://g1_description/urdf/meshes/Link13_L.STL
- added link L_thumb_proximal, mass 0.0066101; collision mesh filename=package://g1_description/urdf/meshes/Link12_L.STL; visual mesh filename=package://g1_description/urdf/meshes/Link12_L.STL
- added link L_thumb_proximal_base, mass 0.0018869; collision mesh filename=package://g1_description/urdf/meshes/Link11_L.STL; visual mesh filename=package://g1_description/urdf/meshes/Link11_L.STL
- added link L_thumb_tip; visual sphere radius=0.005
- added link R_hand_base_link, mass 0.14143; collision mesh filename=package://g1_description/urdf/meshes/R_hand_base_link.STL; visual mesh filename=package://g1_description/urdf/meshes/R_hand_base_link.STL
- added link R_index_intermediate, mass 0.0045683; collision mesh filename=package://g1_description/urdf/meshes/Link16_R.STL; visual mesh filename=package://g1_description/urdf/meshes/Link16_R.STL
- added link R_index_proximal, mass 0.0042403; collision mesh filename=package://g1_description/urdf/meshes/Link15_R.STL; visual mesh filename=package://g1_description/urdf/meshes/Link15_R.STL
- added link R_index_tip; visual sphere radius=0.005
- added link R_middle_intermediate, mass 0.0050396; collision mesh filename=package://g1_description/urdf/meshes/Link18_R.STL; visual mesh filename=package://g1_description/urdf/meshes/Link18_R.STL
- added link R_middle_proximal, mass 0.0042403; collision mesh filename=package://g1_description/urdf/meshes/Link17_R.STL; visual mesh filename=package://g1_description/urdf/meshes/Link17_R.STL
- added link R_middle_tip; visual sphere radius=0.005
- added link R_pinky_intermediate, mass 0.0035996; collision mesh filename=package://g1_description/urdf/meshes/Link22_R.STL; visual mesh filename=package://g1_description/urdf/meshes/Link22_R.STL
- added link R_pinky_proximal, mass 0.0042403; collision mesh filename=package://g1_description/urdf/meshes/Link21_R.STL; visual mesh filename=package://g1_description/urdf/meshes/Link21_R.STL
- added link R_pinky_tip; visual sphere radius=0.005
- added link R_ring_intermediate, mass 0.0045683; collision mesh filename=package://g1_description/urdf/meshes/Link20_R.STL; visual mesh filename=package://g1_description/urdf/meshes/Link20_R.STL
- added link R_ring_proximal, mass 0.0042403; collision mesh filename=package://g1_description/urdf/meshes/Link19_R.STL; visual mesh filename=package://g1_description/urdf/meshes/Link19_R.STL
- added link R_ring_tip; visual sphere radius=0.005
- added link R_thumb_distal, mass 0.0033441; collision mesh filename=package://g1_description/urdf/meshes/Link14_R.STL; visual mesh filename=package://g1_description/urdf/meshes/Link14_R.STL
- added link R_thumb_intermediate, mass 0.0037847; collision mesh filename=package://g1_description/urdf/meshes/Link13_R.STL; visual mesh filename=package://g1_description/urdf/meshes/Link13_R.STL
- added link R_thumb_proximal, mass 0.0066075; collision mesh filename=package://g1_description/urdf/meshes/Link12_R.STL; visual mesh filename=package://g1_description/urdf/meshes/Link12_R.STL
- added link R_thumb_proximal_base, mass 0.0018869; collision mesh filename=package://g1_description/urdf/meshes/Link11_R.STL; visual mesh filename=package://g1_description/urdf/meshes/Link11_R.STL
- added link R_thumb_tip; visual sphere radius=0.005
Joints:
- removed joint left_hand_index_0_joint
- removed joint left_hand_index_1_joint
- removed joint left_hand_middle_0_joint
- removed joint left_hand_middle_1_joint
- removed joint left_hand_palm_joint
- removed joint left_hand_thumb_0_joint
- removed joint left_hand_thumb_1_joint
- removed joint left_hand_thumb_2_joint
- removed joint right_hand_index_0_joint
- removed joint right_hand_index_1_joint
- removed joint right_hand_middle_0_joint
- removed joint right_hand_middle_1_joint
- removed joint right_hand_palm_joint
- removed joint right_hand_thumb_0_joint
- removed joint right_hand_thumb_1_joint
- removed joint right_hand_thumb_2_joint
- added joint L_index_intermediate_joint: type revolute, parent L_index_proximal, child L_index_intermediate, origin xyz=-0.0024229 -0.032041 -0.001 rpy=0 0 0, axis 0 0 -1, limit lower=0 upper=1.7 effort=1 velocity=0.5, mimic joint=L_index_proximal_joint multiplier=1 offset=0
- added joint L_index_proximal_joint: type revolute, parent L_hand_base_link, child L_index_proximal, origin xyz=0.00028533 -0.13653 0.032268 rpy=-0.034907 0 0, axis 0 0 -1, limit lower=0 upper=1.7 effort=1 velocity=0.5
- added joint L_index_tip_joint: type fixed, parent L_index_intermediate, child L_index_tip, origin xyz=-0.005 -0.04 -0.004 rpy=0 0 0
- added joint L_middle_intermediate_joint: type revolute, parent L_middle_proximal, child L_middle_intermediate, origin xyz=-0.0024229 -0.032041 -0.001 rpy=0 0 0, axis 0 0 -1, limit lower=0 upper=1.7 effort=1 velocity=0.5, mimic joint=L_middle_proximal_joint multiplier=1 offset=0
- added joint L_middle_proximal_joint: type revolute, parent L_hand_base_link, child L_middle_proximal, origin xyz=0.00028533 -0.1371 0.01295 rpy=0 0 0, axis 0 0 -1, limit lower=0 upper=1.7 effort=1 velocity=0.5
- added joint L_middle_tip_joint: type fixed, parent L_middle_intermediate, child L_middle_tip, origin xyz=-0.005 -0.045 -0.004 rpy=0 0 0
- added joint L_pinky_intermediate_joint: type revolute, parent L_pinky_proximal, child L_pinky_intermediate, origin xyz=-0.0024229 -0.032041 -0.001 rpy=0 0 0, axis 0 0 -1, limit lower=0 upper=1.7 effort=1 velocity=0.5, mimic joint=L_pinky_proximal_joint multiplier=1 offset=0
- added joint L_pinky_proximal_joint: type revolute, parent L_hand_base_link, child L_pinky_proximal, origin xyz=0.00028533 -0.13571 -0.025488 rpy=0.10472 0 0, axis 0 0 -1, limit lower=0 upper=1.7 effort=1 velocity=0.5
- added joint L_pinky_tip_joint: type fixed, parent L_pinky_intermediate, child L_pinky_tip, origin xyz=-0.002 -0.032 -0.004 rpy=0 0 0
- added joint L_ring_intermediate_joint: type revolute, parent L_ring_proximal, child L_ring_intermediate, origin xyz=-0.0024229 -0.032041 -0.001 rpy=0 0 0, axis 0 0 -1, limit lower=0 upper=1.7 effort=1 velocity=0.5, mimic joint=L_ring_proximal_joint multiplier=1 offset=0
- added joint L_ring_proximal_joint: type revolute, parent L_hand_base_link, child L_ring_proximal, origin xyz=0.00028533 -0.13691 -0.0062872 rpy=0.05236 0 0, axis 0 0 -1, limit lower=0 upper=1.7 effort=1 velocity=0.5
- added joint L_ring_tip_joint: type fixed, parent L_ring_intermediate, child L_ring_tip, origin xyz=-0.002 -0.04 -0.004 rpy=0 0 0
- added joint L_thumb_distal_joint: type revolute, parent L_thumb_intermediate, child L_thumb_distal, origin xyz=0.020248 -0.010156 -0.0012 rpy=0 0 0, axis 0 0 -1, limit lower=0 upper=1.2 effort=1 velocity=0.5, mimic joint=L_thumb_proximal_pitch_joint multiplier=2.4 offset=0
- added joint L_thumb_intermediate_joint: type revolute, parent L_thumb_proximal, child L_thumb_intermediate, origin xyz=0.04407 -0.034553 -0.0008 rpy=0 0 0, axis 0 0 -1, limit lower=0 upper=0.8 effort=1 velocity=0.5, mimic joint=L_thumb_proximal_pitch_joint multiplier=1.6 offset=0
- added joint L_thumb_proximal_pitch_joint: type revolute, parent L_thumb_proximal_base, child L_thumb_proximal, origin xyz=0.0099867 0.0098242 -0.0089 rpy=-1.5708 0 0.16939, axis 0 0 -1, limit lower=0.0 upper=0.5 effort=1 velocity=0.5
- added joint L_thumb_proximal_yaw_joint: type revolute, parent L_hand_base_link, child L_thumb_proximal_base, origin xyz=-0.01696 -0.0691 0.02045 rpy=1.5708 -1.5708 0, axis 0 0 1, limit lower=-0.1 upper=1.3 effort=1 velocity=0.5
- added joint L_thumb_tip_joint: type fixed, parent L_thumb_distal, child L_thumb_tip, origin xyz=0.015 -0.013 -0.004 rpy=0 0 0
- added joint R_index_intermediate_joint: type revolute, parent R_index_proximal, child R_index_intermediate, origin xyz=-0.0026138 0.032026 -0.001 rpy=0 0 0, axis 0 0 1, limit lower=0 upper=1.7 effort=1 velocity=0.5, mimic joint=R_index_proximal_joint multiplier=1 offset=0
- added joint R_index_proximal_joint: type revolute, parent R_hand_base_link, child R_index_proximal, origin xyz=0.00028533 -0.13653 -0.032268 rpy=-3.1067 0 0, axis 0 0 1, limit lower=0 upper=1.7 effort=1 velocity=0.5
- added joint R_index_tip_joint: type fixed, parent R_index_intermediate, child R_index_tip, origin xyz=-0.005 0.04 -0.004 rpy=0 0 0
- added joint R_middle_intermediate_joint: type revolute, parent R_middle_proximal, child R_middle_intermediate, origin xyz=-0.0024229 0.032041 -0.001 rpy=0 0 0, axis 0 0 1, limit lower=0 upper=1.7 effort=1 velocity=0.5, mimic joint=R_middle_proximal_joint multiplier=1 offset=0
- added joint R_middle_proximal_joint: type revolute, parent R_hand_base_link, child R_middle_proximal, origin xyz=0.00028533 -0.1371 -0.01295 rpy=-3.1416 0 0, axis 0 0 1, limit lower=0 upper=1.7 effort=1 velocity=0.5
- added joint R_middle_tip_joint: type fixed, parent R_middle_intermediate, child R_middle_tip, origin xyz=-0.005 0.045 -0.004 rpy=0 0 0
- added joint R_pinky_intermediate_joint: type revolute, parent R_pinky_proximal, child R_pinky_intermediate, origin xyz=-0.0024229 0.032041 -0.001 rpy=0 0 0, axis 0 0 1, limit lower=0 upper=1.7 effort=1 velocity=0.5, mimic joint=R_pinky_proximal_joint multiplier=1 offset=0
- added joint R_pinky_proximal_joint: type revolute, parent R_hand_base_link, child R_pinky_proximal, origin xyz=0.00028533 -0.13571 0.025488 rpy=3.0369 0 0, axis 0 0 1, limit lower=0 upper=1.7 effort=1 velocity=0.5
- added joint R_pinky_tip_joint: type fixed, parent R_pinky_intermediate, child R_pinky_tip, origin xyz=-0.002 0.032 -0.004 rpy=0 0 0
- added joint R_ring_intermediate_joint: type revolute, parent R_ring_proximal, child R_ring_intermediate, origin xyz=-0.0024229 0.032041 -0.001 rpy=0 0 0, axis 0 0 1, limit lower=0 upper=1.7 effort=1 velocity=0.5, mimic joint=R_ring_proximal_joint multiplier=1 offset=0
- added joint R_ring_proximal_joint: type revolute, parent R_hand_base_link, child R_ring_proximal, origin xyz=0.00028533 -0.13691 0.0062872 rpy=3.0892 0 0, axis 0 0 1, limit lower=0 upper=1.7 effort=1 velocity=0.5
- added joint R_ring_tip_joint: type fixed, parent R_ring_intermediate, child R_ring_tip, origin xyz=-0.002 0.04 -0.004 rpy=0 0 0
- added joint R_thumb_distal_joint: type revolute, parent R_thumb_intermediate, child R_thumb_distal, origin xyz=0.020248 0.010156 -0.0012 rpy=0 0 0, axis 0 0 1, limit lower=0 upper=1.2 effort=1 velocity=0.5, mimic joint=R_thumb_proximal_pitch_joint multiplier=2.4 offset=0
- added joint R_thumb_intermediate_joint: type revolute, parent R_thumb_proximal, child R_thumb_intermediate, origin xyz=0.04407 0.034553 -0.0008 rpy=0 0 0, axis 0 0 1, limit lower=0 upper=0.8 effort=1 velocity=0.5, mimic joint=R_thumb_proximal_pitch_joint multiplier=1.6 offset=0
- added joint R_thumb_proximal_pitch_joint: type revolute, parent R_thumb_proximal_base, child R_thumb_proximal, origin xyz=-0.0088099 0.010892 -0.00925 rpy=1.5708 0 2.8587, axis 0 0 1, limit lower=0.0 upper=0.5 effort=1 velocity=0.5
- added joint R_thumb_proximal_yaw_joint: type revolute, parent R_hand_base_link, child R_thumb_proximal_base, origin xyz=-0.01696 -0.0691 -0.02045 rpy=1.5708 -1.5708 0, axis 0 0 -1, limit lower=-0.1 upper=1.3 effort=1 velocity=0.5
- added joint R_thumb_tip_joint: type fixed, parent R_thumb_distal, child R_thumb_tip, origin xyz=0.015 0.013 -0.004 rpy=0 0 0
- added joint left_hand_base_joint: type fixed, parent left_wrist_yaw_link, child L_hand_base_link, origin xyz=0.0415 0.003 0 rpy=0 0 1.5707963
- added joint right_hand_base_joint: type fixed, parent right_wrist_yaw_link, child R_hand_base_link, origin xyz=0.0415 -0.003 0 rpy=3.1415927 0 -1.5707963
- joint left_ankle_pitch_joint: limit lower=-0.87267 upper=0.5236 effort=50 velocity=37 -> lower=-0.87267 upper=0.5236 effort=50 velocity=37.0
- joint left_ankle_roll_joint: limit lower=-0.2618 upper=0.2618 effort=50 velocity=37 -> lower=-0.2618 upper=0.2618 effort=50 velocity=37.0
- joint left_elbow_joint: limit lower=-1.0472 upper=2.0944 effort=25 velocity=37 -> lower=-1.0472 upper=2.0944 effort=25 velocity=37.0
- joint left_shoulder_pitch_joint: limit lower=-3.0892 upper=2.6704 effort=25 velocity=37 -> lower=-3.0892 upper=2.6704 effort=25 velocity=37.0
- joint left_shoulder_roll_joint: limit lower=-1.5882 upper=2.2515 effort=25 velocity=37 -> lower=-1.5882 upper=2.2515 effort=25 velocity=37.0
- joint left_shoulder_yaw_joint: limit lower=-2.618 upper=2.618 effort=25 velocity=37 -> lower=-2.618 upper=2.618 effort=25 velocity=37.0
- joint left_wrist_pitch_joint: limit lower=-1.614429558 upper=1.614429558 effort=5 velocity=22 -> lower=-1.614429558 upper=1.614429558 effort=5 velocity=22.0
- joint left_wrist_roll_joint: limit lower=-1.972222054 upper=1.972222054 effort=25 velocity=37 -> lower=-1.972222054 upper=1.972222054 effort=25 velocity=37.0
- joint left_wrist_yaw_joint: limit lower=-1.614429558 upper=1.614429558 effort=5 velocity=22 -> lower=-1.614429558 upper=1.614429558 effort=5 velocity=22.0
- joint right_ankle_pitch_joint: limit lower=-0.87267 upper=0.5236 effort=50 velocity=37 -> lower=-0.87267 upper=0.5236 effort=50 velocity=37.0
- joint right_ankle_roll_joint: limit lower=-0.2618 upper=0.2618 effort=50 velocity=37 -> lower=-0.2618 upper=0.2618 effort=50 velocity=37.0
- joint right_elbow_joint: limit lower=-1.0472 upper=2.0944 effort=25 velocity=37 -> lower=-1.0472 upper=2.0944 effort=25 velocity=37.0
- joint right_shoulder_pitch_joint: limit lower=-3.0892 upper=2.6704 effort=25 velocity=37 -> lower=-3.0892 upper=2.6704 effort=25 velocity=37.0
- joint right_shoulder_roll_joint: limit lower=-2.2515 upper=1.5882 effort=25 velocity=37 -> lower=-2.2515 upper=1.5882 effort=25 velocity=37.0
- joint right_shoulder_yaw_joint: limit lower=-2.618 upper=2.618 effort=25 velocity=37 -> lower=-2.618 upper=2.618 effort=25 velocity=37.0
- joint right_wrist_pitch_joint: limit lower=-1.614429558 upper=1.614429558 effort=5 velocity=22 -> lower=-1.614429558 upper=1.614429558 effort=5 velocity=22.0
- joint right_wrist_roll_joint: limit lower=-1.972222054 upper=1.972222054 effort=25 velocity=37 -> lower=-1.972222054 upper=1.972222054 effort=25 velocity=37.0
- joint right_wrist_yaw_joint: limit lower=-1.614429558 upper=1.614429558 effort=5 velocity=22 -> lower=-1.614429558 upper=1.614429558 effort=5 velocity=22.0
- joint waist_pitch_joint: limit lower=-0.52 upper=0.52 effort=50 velocity=37 -> lower=-0.52 upper=0.52 effort=50 velocity=37.0
- joint waist_roll_joint: limit lower=-0.52 upper=0.52 effort=50 velocity=37 -> lower=-0.52 upper=0.52 effort=50 velocity=37.0

Commit message: modified config to ignore pc within range and urdf object links

File: g1_description/urdf/g1_body29_hand14.urdf (robot description, URDF)
Before this commit: robot g1, 74 links, 73 joints
Links:
- removed link world
- added link odom
Joints:
- joint floating_base_joint: parent world -> odom

Commit message: update frame_id of the lidar

File: g1_description/urdf/g1_body29_hand14.urdf (robot description, URDF)
Before this commit: robot g1, 74 links, 73 joints
Links:
- removed link mid360_link
- added link livox_frame
Joints:
- joint mid360_joint: child mid360_link -> livox_frame

Commit message: - updated urdf config - added slam odom republisher to use unitree slam to get accurate odometry

File: g1_description/urdf/g1_body29_hand14.urdf (robot description, URDF)
Before this commit: robot g1, 74 links, 73 joints
Links:
- added link pelvis_base
Joints:
- added joint pelvis_base_joint: type fixed, parent pelvis_base, child pelvis, origin xyz=0.0 0.0 0.717677891254425 rpy=0 0 0
- joint floating_base_joint: child pelvis -> pelvis_base
